File: MXMLP-Corne.kicad_pcb (KiCad board)
At the start: 2 copper layers, 275.5 x 105.6 mm, 88 parts, among them J1 Conn_01x04_Female, J2 Conn_01x04_Female, SW1 SW_Push, SW10 SW_Push, SW11 SW_Push, SW12 SW_Push, SW13 SW_Push, SW14 SW_Push, SW15 SW_Push, SW16 SW_Push, SW17 SW_Push, SW18 SW_Push, SW19 SW_Push, SW2 SW_Push, SW20 SW_Push, SW21 SW_Push, SW22 SW_Push, SW23 SW_Push, SW24 SW_Push, SW25 SW_Push, SW26 SW_Push, SW27 SW_Push, SW28 SW_Push, SW29 SW_Push, SW3 SW_Push, SW30 SW_Push, SW31 SW_Push, SW32 SW_Push, SW33 SW_Push, SW34 SW_Push, SW35 SW_Push, SW36 SW_Push, SW37 SW_Push, SW38 SW_Push, SW39 SW_Push, SW4 SW_Push, SW40 SW_Push, SW41 SW_Push, SW42 SW_Push, SW5 SW_Push, SW6 SW_Push, SW7 SW_Push, SW8 SW_Push, SW9 SW_Push, U1 ProMicro, U2 ProMicro

Commit message: Fixed some footprints
Parts:
- added REF**: breakaway-mousebites, Keebio-Parts:breakaway-mousebites, F.Cu at (58.0, 83.8)
- added REF**: breakaway-mousebites, Keebio-Parts:breakaway-mousebites, F.Cu at (19.9, 83.6)
- added REF**: breakaway-mousebites, Keebio-Parts:breakaway-mousebites, F.Cu at (58.0, 21.8)
- added REF**: breakaway-mousebites, Keebio-Parts:breakaway-mousebites, F.Cu at (96.0, 21.9)
- added REF**: breakaway-mousebites, Keebio-Parts:breakaway-mousebites, F.Cu at (276.6, 83.6)
- added REF**: breakaway-mousebites, Keebio-Parts:breakaway-mousebites, F.Cu at (238.8, 83.5)
- added REF**: breakaway-mousebites, Keebio-Parts:breakaway-mousebites, F.Cu at (238.3, 21.8)
- added REF**: breakaway-mousebites, Keebio-Parts:breakaway-mousebites, F.Cu at (200.5, 21.8)
- added U4: HOLE, Keebio-Parts:MountingHole, F.Cu at (267.1, 64.3)
- added U4: HOLE, Keebio-Parts:MountingHole, F.Cu at (29.6, 64.3)
- added U4: HOLE, Keebio-Parts:MountingHole, F.Cu at (267.1, 45.3)
- added U4: HOLE, Keebio-Parts:MountingHole, F.Cu at (191.1, 41.8)
- added U4: HOLE, Keebio-Parts:MountingHole, F.Cu at (224.0, 81.5)
- added U4: HOLE, Keebio-Parts:MountingHole, F.Cu at (177.4, 89.1)
- added U4: HOLE, Keebio-Parts:MountingHole, F.Cu at (119.3, 89.1)
- added U4: HOLE, Keebio-Parts:MountingHole, F.Cu at (72.8, 81.5)
- added U4: HOLE, Keebio-Parts:MountingHole, F.Cu at (105.6, 41.8)
- added U4: HOLE, Keebio-Parts:MountingHole, F.Cu at (29.6, 45.3)
- D1, D10, D11, D12, D13, D14, D15, D16, D17, D18, D19, D2, D20, D21, D22, D23, D24, D25, D26, D27, D28, D29, D3, D30, D31, D32, D33, D34, D35, D36, D37, D38, D39, D4, D40, D41, D42, D5, D6, D7, D8, D9: footprint kbd:D3_SMD_v2 -> Keebio-Parts:Diode-Hybrid-Back; moved to F.Cu
- U1, U2: footprint kbd:ProMicro_v3 -> promicro:ProMicro; moved to B.Cu
- moved U2 27.2 mm to (134.8, 46.1), turned to 270 degrees
- moved U1 27.2 mm to (162.0, 46.0), turned to 270 degrees
- moved D41 17.4 mm to (196.2, 84.9), turned to 105 degrees
- moved D32 15.4 mm to (192.2, 50.1), turned to 90 degrees
- moved D37 15.4 mm to (211.2, 66.4), turned to 90 degrees
- moved D34 15.4 mm to (268.3, 72.4), turned to 90 degrees
- moved D36 15.3 mm to (230.2, 66.6), turned to 90 degrees
- moved D29 15.3 mm to (249.4, 51.2), turned to 90 degrees
- moved D30 15.2 mm to (230.3, 46.7), turned to 90 degrees
- moved D28 15.2 mm to (268.4, 53.8), turned to 90 degrees
- moved D26 15.2 mm to (192.3, 30.8), turned to 90 degrees
- moved D27 15.2 mm to (173.3, 32.9), turned to 90 degrees
- moved D39 15.2 mm to (173.3, 68.3), turned to 90 degrees
- moved D23 15.1 mm to (249.4, 33.2), turned to 90 degrees
- moved D22 15.1 mm to (268.5, 33.3), turned to 90 degrees
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Connections:
- J2 pad 3: GND -> GNDA
- U1 pad 1: LED -> LED_r
- U1 pad 10: row3 -> row3_r
- U1 pad 15: col5 -> col5_r
- U1 pad 16: col4 -> col4_r
- U1 pad 17: col3 -> col3_r
- U1 pad 18: col2 -> col2_r
- U1 pad 19: col1 -> col1_r
- U1 pad 2: data -> data_r
- U1 pad 20: col0 -> col0_r
- U1 pad 21: VCC -> VDD
- U1 pad 22: reset -> reset_r
- U1 pad 23: GND -> GNDA
- U1 pad 3: GND -> GNDA
- U1 pad 4: GND -> GNDA
- U1 pad 5: SDA -> SDA_r
- U1 pad 6: SCL -> SCL_r
- U1 pad 7: row0 -> row0_r
- U1 pad 8: row1 -> row1_r
- U1 pad 9: row2 -> row2_r
- U2 pad 1: LED_r -> LED
- U2 pad 10: row3_r -> row3
- U2 pad 15: col5_r -> col5
- U2 pad 16: col4_r -> col4
- U2 pad 17: col3_r -> col3
- U2 pad 18: col2_r -> col2
- U2 pad 19: col1_r -> col1
- U2 pad 2: data_r -> data
- U2 pad 20: col0_r -> col0
- U2 pad 21: VDD -> VCC
- U2 pad 22: reset_r -> reset
- U2 pad 23: GNDA -> GND
- U2 pad 3: GNDA -> GND
- U2 pad 4: GNDA -> GND
- U2 pad 5: SDA_r -> SDA
- U2 pad 6: SCL_r -> SCL
- U2 pad 7: row0_r -> row0
- U2 pad 8: row1_r -> row1
- U2 pad 9: row2_r -> row2
Routing:
- net GNDA: track 18.8 -> 59.8 mm
- net col5_r: track 107.6 -> 146.5 mm
- net col0: track 178.7 -> 214.9 mm
- net col3_r: track 152.4 -> 188.1 mm
- net col4_r: track 132.2 -> 167.3 mm
- net col4: track 126.6 -> 160.4 mm
- net col5: track 125.9 -> 155.7 mm
- net row2: track 132.9 -> 103.3 mm
- net col1_r: track 162.3 -> 191.2 mm
- net col3: track 151.4 -> 180.0 mm
- net col2_r: track 142.2 -> 169.8 mm
- net row1: track 155.4 -> 128.6 mm, vias 2 -> 0
- net col0_r: track 189.4 -> 213.8 mm, vias 0 -> 1
- net col1: track 167.9 -> 188.4 mm
- net col2: track 145.4 -> 165.7 mm
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